File: Kajimba/Kajimba.kicad_sch (KiCad schematic)
At the start: 17 parts, among them J1 Barrel_Jack, J2 Flow sensor JST, J3 Screen, J4 Pump GND, J5 Button, J6 Conn_01x02_Female, K1 SANYOU_SRD_Form_C, Q1 BC547, SW1 Button, U1 Pico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

Commit message: KiCad PCB Pump v02
Parts:
- removed D1: RED, LED_THT:LED_D5.0mm, symbol Device:LED
- removed D2, D3: 1N4007, Diode_THT:D_DO-41_SOD81_P10.16mm_Horizontal, symbol Diode:1N4007
- removed J1: Barrel_Jack, Connector_BarrelJack:BarrelJack_SwitchcraftConxall_RAPC10U_Horizontal, symbol Connector:Barrel_Jack
- removed J3: Screen, Connector_PinSocket_2.54mm:PinSocket_1x04_P2.54mm_Vertical, symbol Connector:Conn_01x04_Female
- removed J4: Pump GND, Connector_PinSocket_2.54mm:PinSocket_1x01_P2.54mm_Vertical, symbol Connector:Conn_01x01_Female
- removed J5: Button, Connector_PinSocket_2.54mm:PinSocket_1x02_P2.54mm_Vertical, symbol Connector:Conn_01x02_Female
- removed J6: Conn_01x02_Female, Connector_PinSocket_2.54mm:PinSocket_1x02_P2.54mm_Vertical, symbol Connector:Conn_01x02_Female
- removed Q1: BC547, Package_TO_SOT_THT:TO-92_Inline, symbol Transistor_BJT:BC547
- removed U2: LM7805_TO220, Package_TO_SOT_THT:TO-220-3_Vertical, symbol Regulator_Linear:LM7805_TO220
- added D1, D2: S2JTR, Diode_SMD:D_SMB, symbol Diode:S2JTR
- added D3: RED, LED_SMD:LED_0805_2012Metric_Pad1.15x1.40mm_HandSolder, symbol Device:LED
- added J1: Barrel_Jack_Switch, Connector_BarrelJack:BarrelJack_Wuerth_6941xx301002, symbol Connector:Barrel_Jack_Switch
- added J2: Pump, Connector_Phoenix_MSTB:PhoenixContact_MSTBA_2,5_2-G-5,08_1x02_P5.08mm_Horizontal, symbol Connector:Conn_01x02_Male
- added J4: Screen, Connector_JST:JST_EH_B4B-EH-A_1x04_P2.50mm_Vertical, symbol Connector:Conn_01x04_Male
- added J5: Button, Connector_JST:JST_EH_B2B-EH-A_1x02_P2.50mm_Vertical, symbol Connector:Conn_01x02_Male
- added Q1: BSS138, Package_TO_SOT_SMD:SOT-23_Handsoldering, symbol Transistor_FET:BSS138
- added U2: LM78M05, Package_TO_SOT_SMD:TO-252-2, symbol Regulator_Linear:LM78M05_TO252
- C1: footprint Capacitor_THT:CP_Radial_D6.3mm_P2.50mm -> Capacitor_SMD:CP_Elec_10x10.5
- C2: value 1uF -> 470uF; footprint Capacitor_THT:CP_Radial_D5.0mm_P2.50mm -> Capacitor_SMD:CP_Elec_10x10.5
- J3: renamed from J2; value Flow sensor JST -> Flow sensor
- K1: value SANYOU_SRD_Form_C -> Relay
- R1: footprint Resistor_THT:R_Axial_DIN0207_L6.3mm_D2.5mm_P10.16mm_Horizontal -> Resistor_SMD:R_0805_2012Metric_Pad1.20x1.40mm_HandSolder
- SW1: footprint Button_Switch_THT:SW_PUSH-12mm -> Button_Switch_SMD:SW_SPST_TL3305A
Connections:
- net +12V: now also D1.2 (A), J1.1
- net +3.3V: now also J5.1 (Pin_1); no longer K1.5
- net +5V: now also K1.5, D2.1 (K), J4.3 (Pin_3), U2.3 (VO)
- net Button: now also U1.21 (GPIO16), J5.2 (Pin_2); no longer U1.24 (GPIO18)
- net GND: now also R1.2, J1.2, J2.2 (Pin_2), J4.4 (Pin_4), Q1.2 (S), U2.2 (GND)
- net Relay: now also U1.24 (GPIO18), D3.2 (A), Q1.1 (G); no longer U1.21 (GPIO16)
- net SCL: now also J4.1 (Pin_1)
- net SDA: now also J4.2 (Pin_2)
- net at K1.2: now also D2.2 (A), Q1.3 (D)
- net at R1.1: now also D3.1 (K)
- net at C1.1: now also D1.1 (K), U2.1 (VI)
- net at K1.3: now also J2.1 (Pin_1)
- no-connect marks 0 -> 1
Other:
- moved on the sheet: J3, SW1

Commit message: KiCad PCB Pump v03
Parts:
- added D4: S2JTR, Diode_SMD:D_SMB, symbol Diode:S2JTR
- added H1, H2, H3, H4: GND_Pad, MountingHole:MountingHole_2.2mm_M2_Pad, symbol Mechanical:MountingHole_Pad
- added Q2: BSS138, Package_TO_SOT_SMD:SOT-23_Handsoldering, symbol Transistor_FET:BSS138
- added R2: 470, Resistor_SMD:R_0805_2012Metric_Pad1.20x1.40mm_HandSolder, symbol Device:R
- added RV1: R_Potentiometer, Potentiometer_THT:Potentiometer_Bourns_3296W_Vertical, symbol Device:R_Potentiometer
- J3: value Flow sensor -> Sensor
Connections:
- net +12V: now also Q2.3 (D), R2.2; no longer K1.1
- net Button: now also U1.12 (GPIO9); no longer U1.21 (GPIO16)
- net GND: now also D4.2 (A), H1.1, H2.1, H3.1, H4.1, RV1.3
- net Relay: now also U1.26 (GPIO20); no longer U1.24 (GPIO18)
- net Sensor: now also U1.11 (GPIO8); no longer U1.22 (GPIO17)
- new net: R2.1, RV1.1
- new net: D4.1 (K), Q2.1 (G), RV1.2
- new net Pump: K1.1, Q2.2 (S)

Commit message: KiCad PCB Pump v04
Parts:
- removed D2: S2JTR, Diode_SMD:D_SMB, symbol Diode:S2JTR
- removed H1, H2, H3, H4: GND_Pad, MountingHole:MountingHole_2.2mm_M2_Pad, symbol Mechanical:MountingHole_Pad
- removed K1: Relay, Relay_THT:Relay_SPDT_SANYOU_SRD_Series_Form_C, symbol Relay:SANYOU_SRD_Form_C
- removed Q1, Q2: BSS138, Package_TO_SOT_SMD:SOT-23_Handsoldering, symbol Transistor_FET:BSS138
- added D4: RED, LED_SMD:LED_0805_2012Metric_Pad1.15x1.40mm_HandSolder, symbol Device:LED
- added Q1: QM6006D, Package_TO_SOT_SMD:TO-252-2, symbol Transistor_FET:QM6006D
- added R3: 1.5k, Resistor_SMD:R_0805_2012Metric_Pad1.20x1.40mm_HandSolder, symbol Device:R
- J1: value Barrel_Jack_Switch -> Barrel Jack
- R1: renamed from R2; value 470 -> 10k
- RV1: value R_Potentiometer -> Pot
- renumbered D4 to D2, R1 to R2
Connections:
- net +12V: now also D2.1 (K), J2.2 (Pin_2); no longer R1.2
- net +3.3V: now also RV1.3
- net Button: now also U1.14 (GPIO10); no longer U1.12 (GPIO9)
- net GND: now also R1.1, RV1.1, Q1.3 (S), R3.2; no longer D2.2 (A), J2.2 (Pin_2), RV1.3
- net Relay: no longer D3.2 (A)
- net at J2.1 (Pin_1): now also D2.2 (A), Q1.2 (D)
- net LED: now reaches U1.24 (GPIO18)
- net LED: now also D4.2 (A)
- net PWM: now reaches U1.25 (GPIO19)
- net PWM: now also D3.2 (A), R1.2, Q1.1 (G)
- net Analog: now reaches U1.31 (GPIO26_ADC0)
- net Analog: now also RV1.2
- new net: D4.1 (K), R3.1
Other:
- moved on the sheet: D2, D3, J2, J3, J4, J5, R1, R2, RV1, SW1
